File: H0FR70/Design/H0FR70.brd (EAGLE design)
At the start: 34.6 x 30 mm, 39 parts, among them P2 HEXABIT_17.32_NO_P6_P7_P12, Q1 BSS123, Q2 STD36P4LLF6, U2 INA199A2DCKT, X1 XTALL_CSTCE8M00G52

Commit message: Zener was deleted prooerties was changed to 12V 20A
Parts:
- removed D4: BZT52C2V0S-7-F, Hexabitz:SOD-323
- moved R1 0.13 mm to (24.6, 33.3)
Connections:
- net AGND: no longer D4.+
- net N$7: no longer D4.-
Routing:
- net N$7: track 12.6 -> 11.9 mm
Other:
- board text added: "12V max"
- board text added: "12V max."
- board text removed: "40V max"
- board text removed: "40V max."
Changed lines of the file:
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@@
 <?xml version="1.0" encoding="utf-8"?>
 <!DOCTYPE eagle SYSTEM "eagle.dtd">
-<eagle version="9.6.0">
+<eagle version="9.6.1">
 <drawing>
 <settings>
@@
 </layers>
 <board>
+<fusionsync huburn="a.cGVyc29uYWw6dWUyYWRmNjYx" projecturn="a.cGVyc29uYWw6dWUyYWRmNjYxIzIwMTcwOTMwOTU4ODcyMDE" f3durn="urn:adsk.wipprod:dm.lineage:N2REdjOcR3KuyEYRzCluEA" pcbguid="7eb57344-c11a-410f-b86c-eded5a1df137" lastpulledtime="" lastsyncedchangeguid="" latestrevisionid="" lastsyncedrevisionid="" lastboardhashguid="" lastpushedtime="" linktopcb3d="%12"/>
 <plain>
 <text x="47.5112" y="35.7238375" size="1.9304" layer="26" rot="MR0">B</text>
@@
 </polygon>
 <text x="46.718984375" y="43.33646875" size="1.016" layer="21" ratio="10" rot="R120">20A max.</text>
-<text x="23.749" y="43.18" size="1.016" layer="21" ratio="10" rot="R60">40V max.</text>
-<text x="33.02" y="48.133" size="1.27" layer="22" ratio="10" rot="MR0">40V max</text>
+<text x="23.749" y="43.18" size="1.016" layer="21" ratio="10" rot="R60">12V max.</text>
+<text x="33.02" y="48.133" size="1.27" layer="22" ratio="10" rot="MR0">12V max</text>
 <text x="43.053" y="48.133" size="1.27" layer="22" ratio="10" rot="MR0">20A max</text>
 <text x="14.478" y="60.833" size="1.4224" layer="51">Note: This module should be manufactured with 2oz copper to handle 20A current.</text>
@@
 <attribute name="VALUE" x="37.338" y="22.225" size="1.27" layer="27" rot="R270"/>
 </element>
-<element name="R1" library="Hexabitz" package="R-0603" value="270.0R" x="24.638" y="33.401" smashed="yes" rot="R270">
-<attribute name="MFN" value="Yageo" x="24.638" y="33.401" size="1.778" layer="27" rot="R270" display="off"/>
-<attribute name="MPN" value="RC0603FR-07270RL" x="24.638" y="33.401" size="1.778" layer="27" rot="R270" display="off"/>
-<attribute name="NAME" x="26.473671875" y="32.026240625" size="1.016" layer="25" rot="R90"/>
-<attribute name="OCTOPART_URL" value="https://octopart.com/search?q=RC0603FR-07270RL&amp;start=0" x="24.638" y="33.401" size="1.778" layer="27" rot="R270" display="off"/>
-<attribute name="RESISTANCE" value="270.0 Ohm" x="24.638" y="33.401" size="1.778" layer="27" rot="R270" display="off"/>
-<attribute name="TOLERANCE" value="1%" x="24.638" y="33.401" size="1.778" layer="27" rot="R270" display="off"/>
-<attribute name="VALUE" x="22.733" y="34.036" size="1.27" layer="27" rot="R270"/>
+<element name="R1" library="Hexabitz" package="R-0603" value="270.0R" x="24.638" y="33.274" smashed="yes" rot="R270">
+<attribute name="MFN" value="Yageo" x="24.638" y="33.274" size="1.778" layer="27" rot="R270" display="off"/>
+<attribute name="MPN" value="RC0603FR-07270RL" x="24.638" y="33.274" size="1.778" layer="27" rot="R270" display="off"/>
+<attribute name="NAME" x="26.473671875" y="31.899240625" size="1.016" layer="25" rot="R90"/>
+<attribute name="OCTOPART_URL" value="https://octopart.com/search?q=RC0603FR-07270RL&amp;start=0" x="24.638" y="33.274" size="1.778" layer="27" rot="R270" display="off"/>
+<attribute name="RESISTANCE" value="270.0 Ohm" x="24.638" y="33.274" size="1.778" layer="27" rot="R270" display="off"/>
+<attribute name="TOLERANCE" value="1%" x="24.638" y="33.274" size="1.778" layer="27" rot="R270" display="off"/>
+<attribute name="VALUE" x="22.733" y="33.909" size="1.27" layer="27" rot="R270"/>
 </element>
 <element name="U1" library="Hexabitz" package="STM32F091CBU6" value="" x="34.544" y="27.559" smashed="yes" rot="MR270">
@@
 <attribute name="TOLERANCE" value="" x="35.306" y="36.068" size="1.778" layer="27" rot="R270" display="off"/>
 <attribute name="VALUE" x="33.415984375" y="37.605971875" size="1.016" layer="27" rot="R270"/>
-</element>
-<element name="D4" library="Hexabitz" package="SOD-323" value="BZT52C2V0S-7-F" x="32.639" y="35.503" smashed="yes" rot="MR270">
-<attribute name="DESCRIPTION" value="BZT52C2V0S Series 2 V 10 mA Surface Mount Zener Diode - SOD-323" x="32.639" y="35.503" size="1.778" layer="28" rot="MR270" display="off"/>
-<attribute name="MFN" value="Diodes Inc." x="32.639" y="35.503" size="1.778" layer="28" rot="MR270" display="off"/>
-<attribute name="MPN" value="BZT52C2V0S-7-F" x="32.639" y="35.503" size="1.778" layer="28" rot="MR270" display="off"/>
-<attribute name="NAME" x="33.274009375" y="36.77301875" size="0.635009375" layer="34" ratio="10" rot="MR270"/>
-<attribute name="NAME" x="34.03535" y="34.742390625" size="0.88965" layer="26" ratio="11" rot="MR270"/>
-<attribute name="OCTOPART_URL" value="https://octopart.com/bzt52c2v0s-7-f-diodes+inc.-7151792?r=sp" x="32.639" y="35.503" size="1.778" layer="28" rot="MR270" display="off"/>
-<attribute name="VALUE" x="34.48371875" y="37.41133125" size="0.890553125" layer="28" ratio="11" rot="MR270"/>
 </element>
 </elements>
@@
 <wire x1="25.84238125" y1="33.147" x2="26.41638125" y2="32.573" width="0.3556" layer="16"/>
 <via x="25.84238125" y="33.147" extent="1-16" drill="0.35"/>
-<wire x1="25.84238125" y1="33.147" x2="25.60818125" y2="33.3812" width="0.3556" layer="1"/>
-<wire x1="25.60818125" y1="33.3812" x2="25.146" y2="33.3812" width="0.3556" layer="1"/>
+<wire x1="25.84238125" y1="33.147" x2="25.73518125" y2="33.2542" width="0.3556" layer="1"/>
+<wire x1="25.73518125" y1="33.2542" x2="25.146" y2="33.2542" width="0.3556" layer="1"/>
 <wire x1="48.26" y1="35.306" x2="48.26" y2="36.576" width="0.3556" layer="16"/>
 <wire x1="41.021" y1="32.727" x2="40.64" y2="32.346" width="0.3556" layer="16"/>
@@
 <contactref element="U1" pad="P$32"/>
 <contactref element="R1" pad="2"/>
-<wire x1="24.638" y1="32.551" x2="24.666571875" y2="31.905571875" width="0.3556" layer="1"/>
-<wire x1="24.13" y1="31.369" x2="24.666571875" y2="31.905571875" width="0.3556" layer="1"/>
+<wire x1="24.638" y1="32.424" x2="24.6611875" y2="31.9001875" width="0.3556" layer="1"/>
+<wire x1="24.13" y1="31.369" x2="24.6611875" y2="31.9001875" width="0.3556" layer="1"/>
 <via x="24.13" y="31.369" extent="1-16" drill="0.35"/>
 <wire x1="24.13" y1="31.369" x2="24.13" y2="31.16386875" width="0.254" layer="16"/>
@@
 <contactref element="R1" pad="1"/>
 <contactref element="D1" pad="A"/>
-<wire x1="24.638" y1="34.251" x2="24.638" y2="35.572" width="0.3556" layer="1"/>
+<wire x1="24.638" y1="34.124" x2="24.638" y2="35.572" width="0.3556" layer="1"/>
 </signal>
 <signal name="VDDA">
@@
 <contactref element="R6" pad="2"/>
 <wire x1="35.306" y1="35.218" x2="33.362" y2="33.274" width="0.3556" layer="1"/>
-<contactref element="D4" pad="-"/>
-<wire x1="34.251" y1="35.845" x2="34.251" y2="37.973" width="0.3556" layer="16"/>
-<wire x1="32.469" y1="33.274" x2="32.639" y2="33.444" width="0.3556" layer="16"/>
-<wire x1="32.639" y1="33.444" x2="32.639" y2="34.303" width="0.3556" layer="16"/>
-<wire x1="34.251" y1="35.845" x2="32.709" y2="34.303" width="0.3556" layer="16"/>
-<wire x1="32.709" y1="34.303" x2="32.639" y2="34.303" width="0.3556" layer="16"/>
+<wire x1="34.251" y1="37.973" x2="33.8892" y2="37.6112" width="0.3556" layer="16"/>
+<wire x1="33.8892" y1="37.6112" x2="33.8892" y2="36.8218" width="0.3556" layer="16"/>
+<wire x1="33.8892" y1="36.8218" x2="32.8814" y2="35.814" width="0.3556" layer="16"/>
+<wire x1="32.8814" y1="35.814" x2="30.818" y2="35.814" width="0.3556" layer="16"/>
 </signal>
 <signal name="S">
@@
 <wire x1="33.3812" y1="38.913775" x2="32.932" y2="39.362975" width="0.3556" layer="16"/>
 <contactref element="R5" pad="1"/>
-<contactref element="D4" pad="+"/>
 <wire x1="24.892" y1="36.764" x2="26.824" y2="36.764" width="0.3556" layer="16"/>
 <wire x1="26.824" y1="36.764" x2="26.924" y2="36.664" width="0.3556" layer="16"/>
 <wire x1="28.618" y1="36.764" x2="28.518" y2="36.664" width="0.3556" layer="16"/>
 <wire x1="28.518" y1="36.664" x2="26.924" y2="36.664" width="0.3556" layer="16"/>
-<wire x1="28.618" y1="36.764" x2="32.578" y2="36.764" width="0.3556" layer="16"/>
-<wire x1="32.578" y1="36.764" x2="32.639" y2="36.703" width="0.3556" layer="16"/>
-<wire x1="32.639" y1="36.703" x2="33.051975" y2="36.703" width="0.3556" layer="16"/>
-<wire x1="33.051975" y1="36.703" x2="33.3812" y2="37.032225" width="0.3556" layer="16"/>
+<wire x1="33.112975" y1="36.764" x2="33.3812" y2="37.032225" width="0.3556" layer="16"/>
+<wire x1="33.112975" y1="36.764" x2="28.618" y2="36.764" width="0.3556" layer="16"/>
 </signal>
 <signal name="N$8">
@@
 </note>
 <note version="8.3" severity="warning">
+Since Version 8.3, EAGLE supports Fusion synchronisation.
+This feature will not be available in this version and saving
+the document will break the link to the Fusion PCB feature.
+</note>
+<note version="8.3" severity="warning">

Commit message: PDF fixed R8 changed (2k2 -> 1k) BOM modified
Parts:
- B, C, D, R: device Hexabitz:PAD1 -> HEXABITZ_CONNECTION_PARTS:PAD1
- C1, C11, C12, C13, C3, C5, C6, C8, C9: device Hexabitz:C-0603 -> HEXABITZ_RCLS:C-0603
- C10, C2, C4, C7: device Hexabitz:C-0805-POL -> HEXABITZ_RCLS:C-0805-POL
- D1: device Hexabitz:VLMS1300-GS08 -> HEXABITZ_USER_INTERFACE_PARTS:VLMS1300-GS08
- D2: value ORANGE -> Orange; device Hexabitz:VLMS1300-GS08 -> HEXABITZ_USER_INTERFACE_PARTS:VLMS1300-GS08
- D3: device Hexabitz:SOD-323 -> HEXABITZ_RCLS:SOD-323
- FB1: device Hexabitz:FB-TDK_MMZ1608Y300B -> HEXABITZ_RCLS:FB-TDK_MMZ1608Y300B
- Q1: device Hexabitz:SOT23 -> HEXABITZ_RCLS:SOT23
- Q2: device Hexabitz:DPAK-3 -> HEXABITZ_RCLS:DPAK-3
- R1, R10, R12, R2, R3, R4, R5, R6, R8: device Hexabitz:R-0603 -> HEXABITZ_RCLS:R-0603
- R7: device Hexabitz:R2512 -> HEXABITZ_RCLS:R2512
- U1: device Hexabitz:STM32F091CBU6 -> HEXABITZ_ICs:STM32F091CBU6
- U2: device Hexabitz:SOT65P210X110-6N -> HEXABITZ_ICs:SOT65P210X110-6N
- X1: device Hexabitz:XTALL_CSTCE8M00G52 -> HEXABITZ_OTHER_PARTS:XTALL_CSTCE8M00G52
- X2: device con-ptr500:AK500/3 -> HEXABITZ_CONNECTION_PARTS:AK500/3

Commit message: no message
Parts:
- D2: value Orange -> RED
- R8: value 2k2 -> 1k
Changed lines of the file:
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@@
 </layers>
 <board>
-<fusionsync huburn="a.YnVzaW5lc3M6Z21haWwzNTMyMTg" projecturn="a.YnVzaW5lc3M6Z21haWwzNTMyMTgjMjAxOTA5MjMyMTcyMjExMDY" f3durn="urn:adsk.wipprod:dm.lineage:sew10N-4S7Ct2bmrGT97Lw" pcbguid="" lastpulledtime="" lastsyncedchangeguid="" latestrevisionid="dc9f3fee-6cdd-42b4-8716-bbd353acc209" lastsyncedrevisionid="dc9f3fee-6cdd-42b4-8716-bbd353acc209" lastboardhashguid="2d8d3689-180d-8ab5-3f41-4ff3264f0472" lastpushedtime="2020-05-21T21:19:25Z" linktopcb3d="%12"/>
 <plain>
 <text x="47.5112" y="35.7238375" size="1.9304" layer="26" rot="MR0">B</text>
@@
 </element>
 <element name="P2" library="hexabitz_connectors" library_urn="urn:adsk.eagle:library:20064578" package="HEXABIT_17.32_NO_P6_P7_P12" package3d_urn="urn:adsk.eagle:package:20064634/2" value="HEXABIT_17.32_NO_P6_P7_P12" x="34.671" y="34.671" smashed="yes"/>
-<element name="R8" library="HEXABITZ_RCLS" library_urn="urn:adsk.eagle:library:20064561" package="R-0603" package3d_urn="urn:adsk.eagle:package:1435818/3" value="2k2" x="38.608" y="36.068" smashed="yes" rot="R90">
+<element name="R8" library="HEXABITZ_RCLS" library_urn="urn:adsk.eagle:library:20064561" package="R-0603" package3d_urn="urn:adsk.eagle:package:1435818/3" value="1k" x="38.608" y="36.068" smashed="yes" rot="R90">
 <attribute name="MFN" value="Yageo" x="32.131" y="36.068" size="1.016" layer="27" rot="R90" display="off"/>
-<attribute name="MPN" value="RC0603FR-07270RL" x="32.131" y="36.068" size="1.016" layer="27" rot="R90" display="off"/>
+<attribute name="MPN" value="RC0603JR-071KL" x="32.131" y="36.068" size="1.016" layer="27" rot="R90" display="off"/>
 <attribute name="NAME" x="39.103809375" y="32.93160625" size="1.016" layer="25" rot="R90"/>
-<attribute name="OCTOPART_URL" value="https://octopart.com/search?q=RC0603FR-07270RL&amp;start=0" x="32.131" y="36.068" size="1.016" layer="27" rot="R90" display="off"/>
-<attribute name="RESISTANCE" value="270.0 Ohm" x="32.131" y="36.068" size="1.016" layer="27" rot="R90" display="off"/>
+<attribute name="OCTOPART_URL" value="https://octopart.com/rc0603jr-071kl-yageo-55402888?r=sp" x="32.131" y="36.068" size="1.016" layer="27" rot="R90" display="off"/>
+<attribute name="RESISTANCE" value="1k" x="32.131" y="36.068" size="1.016" layer="27" rot="R90" display="off"/>
 <attribute name="TOLERANCE" value="1%" x="32.131" y="36.068" size="1.016" layer="27" rot="R90" display="off"/>
 <attribute name="VALUE" x="40.498015625" y="34.530028125" size="1.016" layer="27" rot="R90"/>
 </element>
-<element name="D2" library="HEXABITZ_USER_INTERFACE_PARTS" library_urn="urn:adsk.eagle:library:20064563" package="VLMS1300-GS08" package3d_urn="urn:adsk.eagle:package:20064571/2" value="Orange" x="36.957" y="35.941" smashed="yes" rot="R180">
+<element name="D2" library="HEXABITZ_USER_INTERFACE_PARTS" library_urn="urn:adsk.eagle:library:20064563" package="VLMS1300-GS08" package3d_urn="urn:adsk.eagle:package:20064571/2" value="RED" x="36.957" y="35.941" smashed="yes" rot="R180">
 <attribute name="MFN" value="Vishay" x="43.053" y="29.464" size="1.016" layer="27" rot="R180" display="off"/>
 <attribute name="MPN" value="VLMO1300-GS08 " x="43.053" y="29.464" size="1.016" layer="27" rot="R180" display="off"/>
@@
 </element>
 <element name="X2" library="HEXABITZ_CONNECTION_PARTS" library_urn="urn:adsk.eagle:library:20064553" package="AK500/3" package3d_urn="urn:adsk.eagle:package:20388955/4" override_package3d_urn="urn:adsk.eagle:package:20407613/3" override_package_urn="urn:adsk.eagle:footprint:9855/1" value="" x="34.671" y="45.212" smashed="yes" rot="R180">
-<attribute name="MF" value="" x="34.671" y="45.212" size="1.778" layer="27" rot="R180" display="off"/>
-<attribute name="MPN" value="" x="34.671" y="45.212" size="1.778" layer="27" rot="R180" display="off"/>
-<attribute name="OC_FARNELL" value="unknown" x="34.671" y="45.212" size="1.778" layer="27" rot="R180" display="off"/>
-<attribute name="OC_NEWARK" value="unknown" x="34.671" y="45.212" size="1.778" layer="27" rot="R180" display="off"/>
-<attribute name="POPULARITY" value="3" x="34.671" y="45.212" size="1.778" layer="27" rot="R180" display="off"/>
+<attribute name="DESCRIPTION" value="Altech 34.403 PCB Terminal, Front wire, 3 Pole, 10.00mm AK500/03DS-10.0-V, 20A, 300V, grey" x="34.671" y="45.212" size="1.778" layer="27" rot="R180" display="off"/>
+<attribute name="MFN" value="Altech" x="34.671" y="45.212" size="1.778" layer="27" rot="R180" display="off"/>
+<attribute name="MPN" value="AK500/3" x="34.671" y="45.212" size="1.778" layer="27" rot="R180" display="off"/>
+<attribute name="OCTOPART_URL" value="https://octopart.com/30.703-altech-46803?r=sp" x="34.671" y="45.212" size="1.778" layer="27" rot="R180" display="off"/>
 <attribute name="VALUE" x="42.2656" y="50.927" size="1.778" layer="27" ratio="10" rot="R180"/>
 </element>
@@
 </note>
 <note version="8.3" severity="warning">
-Since Version 8.3, EAGLE supports Fusion synchronisation.
-This feature will not be available in this version and saving
-the document will break the link to the Fusion PCB feature.
-</note>
-<note version="8.3" severity="warning">
