File: H0FR71/Design/H0FR71.sch (EAGLE design)
At the start: 38 parts, among them P2 HEXABIT_17.32_NO_P6_P7_P12, Q1 BSS123, Q2 STD36P4LLF6, U2 INA199A2DCKT, X1 XTALL_CSTCE8M00G52

Commit message: - Changing the MC with STM32G0 -  Editing the frontend design so it can work at high pwm frequencies
Parts:
- removed B, C, D: PAD1, HEXABITZ_CONNECTION_PARTS:PAD1
- removed C6, C9: 100nF, HEXABITZ_RCLS:C-0603
- removed D3: SMD-DIODE-SCHOTTKY-40V-300MA(SOD-323), HEXABITZ_RCLS:SMD-DIODE-SCHOTTKY-40V-300MA(SOD-323)
- removed Q1: BSS123, HEXABITZ_RCLS:BSS123
- added C14: 1nF, HEXABITZ_RCLS:C-0603
- added D4: DIOD-SOD-123, HEXABITZ_RCLS:DIOD-SOD-123
- added JP2: (no value), pinhead:PINHD-1X3
- added Q3: MMBT3904LT1, HEXABITZ_RCLS:MMBT3904LT1
- added R11, R9: 1K, HEXABITZ_RCLS:R-0603
- added U3: PMD3001D,115, PMD3001D,115:PMD3001DSOT457_NEX
- C1: value 10nF -> 100nF; CAPACITANCE 10nF -> 100nF; MPN C0603C103K5RACTU -> C0603C104K8RACTU; OCTOPART_URL https://octopart.com/c0603c103k5ractu-kemet-133094?r=sp&s=R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 -> https://octopart.com/c0603c104k8ractu-kemet-145075?r=sp&s=9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; VOLTAGE_RATING 50V -> 10V
- C10: value 1.00uF -> 1nF; device HEXABITZ_RCLS:C-0805-POL -> HEXABITZ_RCLS:C-0603; CAPACITANCE 1.00uF -> 100nF; MFN Yageo -> KEMET; MPN CC0805KKX7R7BB105 -> C0603C104K8RACTU; OCTOPART_URL https://octopart.com/cc0805kkx7r7bb105-yageo-8376555?r=sp&s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 -> https://octopart.com/c0603c104k8ractu-kemet-145075?r=sp&s=9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; VOLTAGE_RATING 16V -> 10V
- R: value PAD1 -> (none); device HEXABITZ_CONNECTION_PARTS:PAD1 -> HEXABITZ_USER_INTERFACE_PARTS:PINHD-1X1
- R12: value 10.0K -> 1K
- R4: value 10.0K -> 1k; MPN RC0603JR-0710KL -> RC0603JR-07680KL; OCTOPART_URL https://octopart.com/search?q=RC0603JR-0710KL&start=0 -> https://octopart.com/rc0603jr-07680kl-yageo-40953169?r=sp; RESISTANCE 10.0K Ohm -> 680K Ohm
- R5: value 680K -> 1k
- U1: value (none) -> STM32G0B1CEU6NUFQFPN48_STM32_STM; device HEXABITZ_ICs:STM32F091CBU6 -> HEXABITZ_ICs:STM32G0B1CEU6NUFQFPN48_STM32_STM
Connections:
- removed net B1: B.P$1, R3.2, U1.PF11-OSC_BOOT0
- removed net N$1 (its old number): D.P$1, U1.PA13
- removed net N$2 (its old number): C.P$1, U1.PA14
- removed net R1: C8.1, R.P$1, U1.NRST
- removed net UART1_RX: P2.SD5, U1.PA10
- removed net UART1_TX: P2.SU5, U1.PA9
- new net CLK: JP2.1, JP2.2, R3.2, U1.PA14-BOOT0
- new net DATA: JP2.3, U1.PA13
- new net N$11: Q3.C, R12.1, R4.2, R5.2
- new net N$12: R6.2, U3.E1/E2
- new net N$14: C14.2, Q3.B, R9.1
- new net N$15: C14.1, R11.1
- new net N$5: C8.1, R.1, U1.PF2-NRST
- new net UART4_RX: P2.SD1, U1.PA1
- new net UART4_TX: P2.SU1, U1.PA0
- net +LOAD: now also D4.C
- net AGND: now also C1.2, C2.-, C5.2, C7.-, D4.A, Q3.E, U1.VSS/VSSA, U3.C2, U3.C2_2; no longer C10.-, Q1.S, R5.1
- net CURRENT_SENSE: now also U1.PB12; no longer U1.PA0
- net EN_PIN: now also R11.2, R9.2, U1.PB6; no longer D3.C, R12.2, U1.PB0
- net GND: now also U1.EPAD, U1.PB0, U1.PB1, U1.PB7, U1.PB8, U1.PB9, U1.VSS; no longer C1.2, C2.-, C5.2, C6.2, C7.-, C9.2, U1.EP, U1.PA15, U1.PA6, U1.PB14, U1.PC13, U1.VSS_0, U1.VSS_1, U1.VSS_2, U1.VSS_A
- net N$13: now also C10.1, R4.1; no longer C10.+, D3.A, Q1.G, R12.1, R5.2
- net N$3: now also U1.PB13; no longer U1.PA11
- net N$7: now also C10.2, R5.1, U3.B1/B2; no longer Q1.D, R4.2, R6.2
- net UART5_RX: now also P2.SD5, U1.PD2; no longer P2.SD1, U1.PB4
- net UART5_TX: now also P2.SU5, U1.PD3; no longer P2.SU1, U1.PB3
- net VDD: no longer C5.1, C6.1, C7.+, C9.1, U1.VBAT, U1.VDD_0, U1.VDD_1
- net VDDA: now also C5.1, C7.+, U1.VBAT, U1.VDD/VDDA, U1.VREF+; no longer U1.VDDA
- net V_LOAD: now also R12.2, U3.C1, U3.C1_2; no longer R4.1
Other:
- note added: "BOOT"
- note added: "H0FR71"
- note added: "H0FR71_Backend"
- note added: "H0FR71_Frontend"
- note added: "Ibrahim Zaeiter"
- note added: "SPST MOSFET Switch 20A 18V"
- note added: "V_load=(3.3-18)"
- note added: "Vref Coupling"
- note removed: "0"
- note removed: "Amir Tabbakh"
- note removed: "H0FR7"
- note removed: "H0FR7_Backend"
- note removed: "H0FR7_Frontend"
- note removed: "SPST MOSFET Switch 20A 12V"
- note removed: "VBAT"
- note removed: "VDD Coupling"
- note removed: "V_load=(3.3-12)"
- moved on the sheet: C1, C2, C3, C4, C5, C7, C8, D1, D2, R1, R12, R3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

Commit message: -Correcting some documentaion issues
Other:
- note added: "V_load=(3.3-18) Volts"
- note removed: "V_load=(3.3-18)"
Changed lines of the file:
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@@
 <text x="21.59" y="107.95" size="2.1844" layer="150">Power and Load Connector</text>
 <text x="189.23" y="102.87" size="1.778" layer="150">Gain = 100 V/V</text>
-<text x="143.51" y="168.91" size="1.778" layer="150">V_load=(3.3-18)</text>
+<text x="144.78" y="186.69" size="1.778" layer="150">V_load=(3.3-18) Volts</text>
 </plain>
 <instances>
