File: H0FR72/Design/H0FR72.brd (EAGLE design)
At the start: 34.6 x 30 mm, 43 parts, among them P2 HEXABIT_17.32_NO_P6_P7_P12, Q2 STD36P4LLF6, Q3 MMBT3904LT1, U1 STM32G0B1CEU6N, U2 INA199A2DCKT, U3 PMD3001D,115, X1 XTALL_CSTCE8M00G52

Commit message: -Add additional 10u capacitor to gate driver IC supply
Parts:
- added C17: C-0805, HEXABITZ_RCLS:C-0805
Connections:
- net +VS: now also C17.1
- net VSSA: now also C17.2
Changed lines of the file:
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@@
 <drawing>
 <settings>
-<setting alwaysvectorfont="no"/>
+<setting alwaysvectorfont="yes"/>
 <setting verticaltext="up"/>
 </settings>
@@
 <text x="14.614" y="14.91" size="1.27" layer="21" font="vector" rot="R270" align="center">3V3</text>
 <text x="14.35781875" y="14.938778125" size="1.27" layer="22" font="vector" rot="MR90" align="center">GND</text>
-<text x="7.209" y="2.365" size="1.27" layer="21" font="vector" rot="R35" align="center">3V3</text>
+<text x="9.77985" y="3.656690625" size="1.27" layer="21" font="vector" rot="R60" align="center">3V3</text>
 <text x="-7.355075" y="2.33919375" size="1.27" layer="22" font="vector" rot="MR35" align="center">GND</text>
 <text x="-7.311" y="2.365" size="1.27" layer="21" font="vector" rot="R325" align="center">3V3</text>
@@
 <attribute name="WORKING-VOLTAGE-VDE" value="250V (AC)" x="0.127" y="25.654" size="1.27" layer="27" rot="R180" display="off"/>
 </element>
+<element name="C17" library="HEXABITZ_RCLS" library_urn="urn:adsk.eagle:library:20064561" package="C-0805" package3d_urn="urn:adsk.eagle:package:19666489/3" value="C-0805" x="5.461" y="3.175" smashed="yes">
+<attribute name="CAPACITANCE" value="10uF" x="5.461" y="3.175" size="1.778" layer="27" display="off"/>
+<attribute name="MFN" value="" x="5.461" y="3.175" size="1.778" layer="27" display="off"/>
+<attribute name="MPN" value="GRM21BR6YA106ME43K" x="5.461" y="3.175" size="1.778" layer="27" display="off"/>
+<attribute name="NAME" x="4.572" y="1.397" size="0.8128" layer="25"/>
+<attribute name="OCTOPART_URL" value="" x="5.461" y="3.175" size="1.778" layer="27" display="off"/>
+<attribute name="TOLERANCE" value="" x="5.461" y="3.175" size="1.778" layer="27" display="off"/>
+<attribute name="VALUE" x="4.191" y="0.635" size="1.27" layer="27"/>
+<attribute name="VOLTAGE_RATING" value="35v" x="5.461" y="3.175" size="1.778" layer="27" display="off"/>
+</element>
 </elements>
 <signals>
@@
 <vertex x="-3.72935" y="2.625284375"/>
 <vertex x="-2.5541125" y="3.683"/>
-<vertex x="1.552221875" y="3.683"/>
-<vertex x="2.8749875" y="2.6007375"/>
-<vertex x="2.286" y="2.159"/>
+<vertex x="1.32644375" y="3.683"/>
+<vertex x="2.4939875" y="2.7277375"/>
+<vertex x="1.9558" y="2.3241"/>
 <vertex x="0.508" y="3.048"/>
 <vertex x="-1.397" y="2.667"/>
@@
 <contactref element="C9" pad="2"/>
 <contactref element="C12" pad="2"/>
-<contactref element="C15" pad="2"/>
 <contactref element="C16" pad="2"/>
 <contactref element="Q2" pad="3"/>
@@
 <polygon width="0.1524" layer="1" thermals="no">
 <vertex x="3.937" y="7.112"/>
-<vertex x="3.937" y="3.937"/>
-<vertex x="5.461" y="3.937"/>
+<vertex x="3.937" y="2.413"/>
+<vertex x="5.461" y="2.413"/>
 <vertex x="5.461" y="6.604"/>
 <vertex x="6.477" y="7.62"/>
@@
 <vertex x="6.985" y="4.699"/>
 </polygon>
+<contactref element="C17" pad="1"/>
+<contactref element="C15" pad="2"/>
 </signal>
 <signal name="VSSA">
@@
 <contactref element="C9" pad="1"/>
 <contactref element="C12" pad="1"/>
-<contactref element="C15" pad="1"/>
 <contactref element="C16" pad="1"/>
 <contactref element="C2" pad="2"/>
@@
 <polygon width="0.1524" layer="1" thermals="no" rank="3">
 <vertex x="5.715" y="6.477"/>
-<vertex x="5.715" y="3.81"/>
-<vertex x="8.636" y="3.81"/>
+<vertex x="5.715" y="2.413"/>
+<vertex x="7.239" y="2.413"/>
 <vertex x="8.763" y="3.937"/>
 <vertex x="8.763" y="8.382"/>
@@
 <via x="-10.414" y="17.145" extent="1-16" drill="0.3" diameter="0.55"/>
 <via x="-14.859" y="18.034" extent="1-16" drill="0.3" diameter="0.55"/>
+<contactref element="C17" pad="2"/>
+<contactref element="C15" pad="1"/>
 </signal>
 <signal name="N$12">

Commit message: Design modification
Parts:
- removed C16: (no value), HEXABITZ_RCLS:C-0402
- removed C17: C-0805, HEXABITZ_RCLS:C-0805
- removed J1: (no value), HEXABITZ_CONNECTION_PARTS:691213710003
- removed R8: 1k, HEXABITZ_RCLS:R-0402
- removed U2: INA199A2DCKT, HEXABITZ_ICs:SOT65P210X110-6N
- added D3: DIOD-SOD-123, HEXABITZ_RCLS:SOD123
- added D5: MMSZ4705T1G, HEXABITZ_RCLS:SOD3716X135N
- added D6: V8PAM10S-M3_H, HEXABITZ_RCLS:V8PAM10SHM3H
- added IC1: TSV772IYDT, HEXABITZ_ICs:SOIC127P600X175-8N
- added LOAD, SUPPLY: (no value), HEXABITZ_CONNECTION_PARTS:1546111-2
- added R14: 10k, HEXABITZ_RCLS:R-0402
- added R15: 50k, HEXABITZ_RCLS:R-0402
- added TRIMBLE-LOGO1, TRIMBLE-LOGO2: HEXA-LOGO, HEXABITZ_USER_INTERFACE_PARTS:HEXA-LOGO
- C10: value 1nF -> 10nF
- C11: value 100nF -> 10nF
- C15: value (none) -> ESH477M035AH3AA; device HEXABITZ_RCLS:C-0402 -> HEXABITZ_RCLS:CAPPRD500W60D1000H1700
- C5: device HEXABITZ_RCLS:C-0402 -> HEXABITZ_RCLS:C-0603
- C6: value ESH477M035AH3AA -> 4.7uF; device HEXABITZ_RCLS:CAPPRD500W60D1000H1700 -> HEXABITZ_RCLS:C-0603-POL
- C7: value 4.7uF -> 100nF; device HEXABITZ_RCLS:C-0603-POL -> HEXABITZ_RCLS:C-0402
- C8: value 100nF -> (none)
- D1: device HEXABITZ_USER_INTERFACE_PARTS:VLMS1300-GS08 -> Hexabitz:VLMS1300-GS08
- D2: value ORANGE -> BOURNS_CDSOD323-T03SCBOURNS_CDSOD323-T03SC_0_0; device HEXABITZ_USER_INTERFACE_PARTS:VLMS1300-GS08 -> HEXABITZ_RCLS:BOURNS_CDSOD323-T03SC_0
- FB1: value FB-TDK_MMZ1608Y300B -> (none); device HEXABITZ_RCLS:FB-TDK_MMZ1608Y300B -> HEXABITZ_RCLS:FB-0603
- R1: value 270.0R -> 270R; device HEXABITZ_RCLS:R-0402 -> HEXABITZ_RCLS:R-0603
- R10, R13: value 10R -> 1k
- R11: value 1K -> 47
- R12: value 1K -> 10k
- R2: device HEXABITZ_RCLS:R-0402 -> HEXABITZ_RCLS:R-0603
- R3: value 10.0K -> 10k
- R4: value 1k -> 10
- R5: value 1k -> 150
- R6: value 10R -> 50k
- R7: value 0.001R -> 2.5m; device HEXABITZ_RCLS:R1206 -> HEXABITZ_RCLS:R2512
- R9: value 1K -> 3.3k
- moved D4 89.2 mm to (-7.87, -65.0), flipped to the top
- moved C13 78.7 mm to (-19.7, -59.7), turned to 0 degrees
- moved C12 74.7 mm to (-19.7, -51.9)
- moved C11 73.7 mm to (-19.7, -55.1), turned to 0 degrees
- moved C8 65.2 mm to (-19.7, -48.8), flipped to the top
- moved C10 57.9 mm to (-19.7, -44.2), flipped to the top, turned to 0 degrees
- moved R7 50.9 mm to (-17.1, -31.0), turned to 0 degrees
- moved R6 50.5 mm to (-19.6, -36.4), turned to 0 degrees
- moved C6 38.2 mm to (-6.86, -16.3), flipped to the top
- moved D2 37.8 mm to (-6.22, -12.7), turned to 0 degrees
- moved D1 34.4 mm to (-14.9, -14.2)
- moved C5 30.2 mm to (-11.7, -19.8), flipped to the top
- moved R2 26.8 mm to (3.17, -4.70), flipped to the top, turned to 0 degrees
- moved FB1 26.3 mm to (-3.05, -9.27), turned to 0 degrees
- moved R1 22.5 mm to (-1.52, -4.70), flipped to the top, turned to 0 degrees
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Connections:
- removed net +LOAD: D4.2, J1.3, R13.2, R7.2, R8.2
- removed net CS: Q2.4, R10.2, R7.1
- removed net EN_PIN: R11.2, R9.2, U1.39
- removed net N$10: Q2.1, R6.1
- removed net N$11: C13.1, R10.1, U2.4
- removed net N$12: R6.2, U3.4
- removed net N$18: C13.2, R13.1, U2.5
- removed net N$7: C10.2, R5.1, U3.1
- new net AGND: C5.2, C6.2, R2.2
- new net LED_INDICATOR: R1.1, U1.15
- new net LOAD+: D6.1, LOAD.1, Q2.4
- new net LOAD-: LOAD.2, R10.2, R7.2
- new net N$19: D3.2, D5.2, Q2.1, R14.2, R5.1
- new net N$6: C11.1, IC1.3, R10.1, R6.2
- new net N$9: C10.1, IC1.2, R13.1, R15.2
- new net SWITCH_CONTROL: R11.2, R9.2, U1.28
- new net VCC: C13.2, IC1.8
- net +VS: now also C15.1, C8.2, D4.1, R14.1, SUPPLY.1; no longer C15.2, C16.2, C17.1, C6.1, J1.1
- net CURRENT_SENSE: now also C10.2, IC1.1, R15.1; no longer U2.6
- net GND: now also C7.2, D2.2; no longer C8.2
- net N$13: now also D3.1; no longer C10.1
- net N$16: now also U3.4; no longer Q3.3, R12.1
- net N$3: now also Q3.3, R12.1, U3.1; no longer R1.2, U1.15
- net N$4: now also R1.2; no longer R1.1
- net N$5: now also C7.1; no longer C8.1
- net N$8: now also D4.2, D5.1; no longer D2.A, R8.1
- net VDD: now also D2.1, FB1.1; no longer FB1.2
- net VDDA: now also C6.1, FB1.2; no longer C11.1, C7.1, FB1.1, U2.3
- net VSSA: now also C13.1, C15.2, C8.1, D6.2, IC1.4, R13.2, R6.1, R7.1, SUPPLY.2; no longer C15.1, C16.1, C17.2, C5.2, C6.2, C7.2, D2.C, D4.1, J1.2, R2.2, U2.1, U2.2
Routing:
- net VDDA: track 13.9 -> 2.24 mm, vias 1 -> 0
- net GND: track 8.52 -> 2.73 mm, vias 11 -> 10
- net +LOAD: track 3.80 -> 0.00 mm
- net EN_PIN: track 3.51 -> 0.00 mm
- net SWITCH_CONTROL: track 0.00 -> 3.51 mm
- net N$3: track 2.23 -> 0.00 mm
- net LED_INDICATOR: track 0.00 -> 2.09 mm
- net N$16: track 4.32 -> 2.47 mm
- net N$8: track 1.83 -> 0.00 mm, vias 1 -> 0
- net N$4: track 1.66 -> 0.00 mm, vias 1 -> 0
- net N$7: track 1.59 -> 0.00 mm, vias 3 -> 2
- net N$13: track 0.73 -> 0.00 mm
- added copper zone on layer 1, net LOAD+
- added copper zone on layer 16, net LOAD+
- removed copper zone on layer 1, net +LOAD
- removed copper zone on layer 16, net +LOAD

Commit message: Design modification
Parts:
- removed R15: 50k, HEXABITZ_RCLS:R-0402
- added R8: 49.9k, HEXABITZ_RCLS:R-0402
- C2: value 1.00uF -> 1uF
- R6: value 50k -> 49.9k
- moved R7 55.9 mm to (22.5, 8.38)
- moved C11 42.3 mm to (14.5, -30.1)
- moved C12 42.3 mm to (14.5, -26.9)
- moved C13 42.3 mm to (14.5, -34.7)
- moved C8 42.3 mm to (14.5, -23.7)
- moved D4 38.4 mm to (6.73, -29.5)
- moved D5 38.4 mm to (6.48, -25.3)
- moved C10 35.5 mm to (-10.2, -10.0)
- moved R6 35.5 mm to (-10.0, -2.29)
- renumbered IC1 to U2, P2 to P1, Q3 to Q1
Connections:
- removed net AGND: C5.2, C6.2, R2.2
- net CURRENT_SENSE: now also R8.1; no longer R15.1
- net N$9: now also R8.2; no longer R15.2
- net VSSA: now also C5.2, C6.2, R2.2
Routing:
- net CLK: track 18.0 -> 16.3 mm

Commit message: Schematic modification
Parts:
- added R15: 100k, HEXABITZ_RCLS:R-0402
Connections:
- net N$14: now also R15.1
- net VSSA: now also R15.2
Changed lines of the file:
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@@
 <attribute name="VALUE" x="6.477" y="-25.273" size="1.27" layer="27" align="center"/>
+</element>
+<element name="R15" library="HEXABITZ_RCLS" library_urn="urn:adsk.eagle:library:20064561" package="R-0402" package3d_urn="urn:adsk.eagle:package:19666455/3" value="100k" x="-16.002" y="4.445" smashed="yes">
+<attribute name="MFN" value="Yageo" x="-16.002" y="4.445" size="1.778" layer="27" display="off"/>
+<attribute name="MPN" value="RC0603JR-07680KL" x="-16.002" y="4.445" size="1.778" layer="27" display="off"/>
+<attribute name="NAME" x="-17.15008125" y="5.0698375" size="0.762" layer="25"/>
+<attribute name="OCTOPART_URL" value="https://octopart.com/rc0603jr-07680kl-yageo-40953169?r=sp" x="-16.002" y="4.445" size="1.778" layer="27" display="off"/>
+<attribute name="RESISTANCE" value="680K Ohm" x="-16.002" y="4.445" size="1.778" layer="27" display="off"/>
+<attribute name="TOLERANCE" value="5%" x="-16.002" y="4.445" size="1.778" layer="27" display="off"/>
+<attribute name="VALUE" x="-17.147540625" y="3.020059375" size="0.762" layer="27"/>
 </element>
 </elements>
@@
 <wire x1="1.694" y1="4.384" x2="0.33" y2="4.384" width="0.6096" layer="16"/>
 <wire x1="0.33" y1="4.384" x2="0.269" y2="4.445" width="0.6096" layer="16"/>
+<contactref element="R15" pad="1"/>
+<wire x1="0.269" y1="4.064" x2="-16.652" y2="4.445" width="0" layer="19" extent="1-16"/>
 </signal>
 <signal name="N$15">
@@
 <contactref element="C6" pad="2"/>
 <contactref element="C15" pad="2"/>
-<wire x1="15.128" y1="-30.099" x2="13.828" y2="-34.671" width="0" layer="19" extent="1-1"/>
-<wire x1="13.828" y1="-26.924" x2="15.128" y2="-30.099" width="0" layer="19" extent="1-1"/>
-<wire x1="13.828" y1="-23.749" x2="13.828" y2="-26.924" width="0" layer="19" extent="1-1"/>
-<wire x1="-10.683" y1="-2.286" x2="13.828" y2="-23.749" width="0" layer="19" extent="1-1"/>
-<wire x1="19.679" y1="8.382" x2="-10.683" y2="-2.286" width="0" layer="19" extent="1-1"/>
-<wire x1="-11.464" y1="-24.892" x2="19.679" y2="8.382" width="0" layer="19" extent="1-1"/>
+<contactref element="R15" pad="2"/>
+<wire x1="-11.464" y1="-24.892" x2="-15.352" y2="4.445" width="0" layer="19" extent="1-1"/>
 <wire x1="-10.834" y1="-19.812" x2="-11.464" y2="-24.892" width="0" layer="19" extent="1-1"/>
 <wire x1="-6.008" y1="-16.256" x2="-10.834" y2="-19.812" width="0" layer="19" extent="1-1"/>
 <wire x1="-2.712" y1="-22.352" x2="-6.008" y2="-16.256" width="0" layer="19" extent="1-1"/>
-<wire x1="4.025" y1="-4.699" x2="-6.008" y2="-16.256" width="0" layer="19" extent="1-1"/>
-<wire x1="7.889" y1="4.191" x2="4.025" y2="-4.699" width="0" layer="19" extent="1-16"/>
-<wire x1="8.382" y1="5.207" x2="7.889" y2="4.191" width="0" layer="19" extent="16-16"/>
-<wire x1="7.1946" y1="6.858" x2="8.382" y2="5.207" width="0" layer="19" extent="1-1"/>
-<wire x1="7.1946" y1="7.808" x2="7.1946" y2="6.858" width="0" layer="19" extent="1-1"/>
-<wire x1="7.62" y1="8.255" x2="7.1946" y2="7.808" width="0" layer="19" extent="1-1"/>
-<wire x1="1.694" y1="6.284" x2="7.1946" y2="6.858" width="0" layer="19" extent="1-16"/>
-<wire x1="7.62" y1="15.748" x2="7.62" y2="8.255" width="0" layer="19" extent="1-1"/>
-<wire x1="7.62" y1="16.51" x2="7.62" y2="15.748" width="0" layer="19" extent="1-1"/>
-<wire x1="9.779" y1="20.828" x2="7.62" y2="16.51" width="0" layer="19" extent="1-1"/>
-<wire x1="9.652" y1="21.463" x2="9.779" y2="20.828" width="0" layer="19" extent="1-1"/>
-<wire x1="-4.142" y1="11.8071" x2="1.694" y2="6.284" width="0" layer="19" extent="16-16"/>
-<wire x1="-7.508" y1="7.747" x2="-7.49293125" y2="10.033" width="0" layer="19" extent="16-16"/>
-<wire x1="-7.708" y1="6.858" x2="-7.508" y2="7.747" width="0" layer="19" extent="16-16"/>
+<wire x1="-10.683" y1="-2.286" x2="-6.008" y2="-16.256" width="0" layer="19" extent="1-1"/>
+<wire x1="-7.708" y1="6.858" x2="-10.683" y2="-2.286" width="0" layer="19" extent="1-16"/>
+<wire x1="-7.508" y1="7.747" x2="-7.708" y2="6.858" width="0" layer="19" extent="16-16"/>
+<wire x1="-7.49293125" y1="10.033" x2="-7.508" y2="7.747" width="0" layer="19" extent="16-16"/>
 <wire x1="-10.414" y1="17.145" x2="-7.49293125" y2="10.033" width="0" layer="19" extent="16-16"/>
 <wire x1="-10.16" y1="19.939" x2="-10.414" y2="17.145" width="0" layer="19" extent="1-1"/>
@@
 <wire x1="-14.859" y1="18.034" x2="-10.414" y2="17.145" width="0" layer="19" extent="1-1"/>
 <wire x1="-0.047" y1="20.066" x2="-6.589" y2="19.685" width="0" layer="19" extent="1-1"/>
-<wire x1="23.368" y1="-0.127" x2="8.382" y2="5.207" width="0" layer="19" extent="1-1"/>
+<wire x1="1.694" y1="6.284" x2="-4.142" y2="11.8071" width="0" layer="19" extent="16-16"/>
+<wire x1="7.1946" y1="6.858" x2="1.694" y2="6.284" width="0" layer="19" extent="1-16"/>
+<wire x1="7.1946" y1="7.808" x2="7.1946" y2="6.858" width="0" layer="19" extent="1-1"/>
+<wire x1="7.62" y1="8.255" x2="7.1946" y2="7.808" width="0" layer="19" extent="1-1"/>
+<wire x1="8.382" y1="5.207" x2="7.1946" y2="6.858" width="0" layer="19" extent="1-1"/>
+<wire x1="7.889" y1="4.191" x2="8.382" y2="5.207" width="0" layer="19" extent="16-16"/>
+<wire x1="7.62" y1="15.748" x2="7.62" y2="8.255" width="0" layer="19" extent="1-1"/>
+<wire x1="7.62" y1="16.51" x2="7.62" y2="15.748" width="0" layer="19" extent="1-1"/>
+<wire x1="9.779" y1="20.828" x2="7.62" y2="16.51" width="0" layer="19" extent="1-1"/>
+<wire x1="9.652" y1="21.463" x2="9.779" y2="20.828" width="0" layer="19" extent="1-1"/>
+<wire x1="4.025" y1="-4.699" x2="7.889" y2="4.191" width="0" layer="19" extent="1-16"/>
+<wire x1="19.679" y1="8.382" x2="8.382" y2="5.207" width="0" layer="19" extent="1-1"/>
+<wire x1="23.368" y1="-0.127" x2="19.679" y2="8.382" width="0" layer="19" extent="1-1"/>
+<wire x1="13.828" y1="-23.749" x2="-2.712" y2="-22.352" width="0" layer="19" extent="1-1"/>
+<wire x1="13.828" y1="-26.924" x2="13.828" y2="-23.749" width="0" layer="19" extent="1-1"/>
+<wire x1="15.128" y1="-30.099" x2="13.828" y2="-26.924" width="0" layer="19" extent="1-1"/>
+<wire x1="13.828" y1="-34.671" x2="15.128" y2="-30.099" width="0" layer="19" extent="1-1"/>
 </signal>
 <signal name="N$12">

Commit message: -Edit the description
Routing:
- net LOAD+: track 0.00 -> 13.4 mm
Changed lines of the file:
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@@
 <contactref element="Q2" pad="4"/>
 <contactref element="D6" pad="1"/>
+<wire x1="-2.794" y1="12.6365" x2="-2.794" y2="18.02659375" width="5.08" layer="1"/>
+<wire x1="-2.794" y1="18.02659375" x2="-3.4315" y2="18.66409375" width="5.08" layer="1"/>
+<wire x1="-3.4315" y1="25.4025" x2="-3.683" y2="25.654" width="5.08" layer="1"/>
+<wire x1="-3.4315" y1="18.66409375" x2="-3.4315" y2="25.4025" width="5.08" layer="1"/>
 <wire x1="18.288" y1="-11.43" x2="-14.684" y2="-24.892" width="0" layer="19" extent="1-1"/>
 <wire x1="-2.794" y1="12.6365" x2="18.288" y2="-11.43" width="0" layer="19" extent="1-1"/>
@@
 <wire x1="-6.589" y1="19.685" x2="-10.16" y2="19.939" width="0" layer="19" extent="1-1"/>
 <wire x1="-14.859" y1="18.034" x2="-10.414" y2="17.145" width="0" layer="19" extent="1-1"/>
-<wire x1="-0.047" y1="20.066" x2="-6.589" y2="19.685" width="0" layer="19" extent="1-1"/>
+<wire x1="-6.589" y1="19.685" x2="-0.047" y2="20.066" width="0" layer="19" extent="1-1"/>
 <wire x1="1.694" y1="6.284" x2="-4.142" y2="11.8071" width="0" layer="19" extent="16-16"/>
 <wire x1="7.1946" y1="6.858" x2="1.694" y2="6.284" width="0" layer="19" extent="1-16"/>
