File: H0FR72/Design/H0FR72.sch (EAGLE design)
At the start: 44 parts, among them P2 HEXABIT_17.32_NO_P6_P7_P12, Q2 STD36P4LLF6, Q3 MMBT3904LT1, U1 STM32G0B1CEU6N, U2 INA199A2DCKT, U3 PMD3001D,115, X1 XTALL_CSTCE8M00G52

Commit message: Design modification
Parts:
- removed C16: (no value), HEXABITZ_RCLS:C-0402
- removed C17: C-0805, HEXABITZ_RCLS:C-0805
- removed J1: (no value), HEXABITZ_CONNECTION_PARTS:691213710003
- removed R8: 1k, HEXABITZ_RCLS:R-0402
- removed U2: INA199A2DCKT, HEXABITZ_ICs:INA199A2DCKT
- added D3: DIOD-SOD-123, HEXABITZ_RCLS:DIOD-SOD-123
- added D5: MMSZ4705T1G, HEXABITZ_RCLS:MMSZ4705T1G
- added D6: V8PAM10S-M3_H, HEXABITZ_RCLS:V8PAM10S-M3_H
- added IC1: TSV772IYDT, HEXABITZ_ICs:TSV772IYDT
- added LOAD, SUPPLY: (no value), HEXABITZ_CONNECTION_PARTS:1546111-2
- added R14: 10k, HEXABITZ_RCLS:R-0402
- added R15: 50k, HEXABITZ_RCLS:R-0402
- added TRIMBLE-LOGO1, TRIMBLE-LOGO2: HEXA-LOGO, HEXABITZ_USER_INTERFACE_PARTS:HEXA-LOGO
- C10: value 1nF -> 10nF; TOLERANCE 10% -> 10V; VOLTAGE_RATING 10V -> 10%
- C11: value 100nF -> 10nF
- C15: value (none) -> ESH477M035AH3AA; device HEXABITZ_RCLS:C-0402 -> HEXABITZ_RCLS:ESH477M035AH3AA; CAPACITANCE 100nF -> 470uF; VOLTAGE_RATING 50V -> (none); VOLT_RATING (none) -> 35V
- C5: device HEXABITZ_RCLS:C-0402 -> HEXABITZ_RCLS:C-0603; CAPACITANCE 100nF -> (none); MFN KEMET -> (none); MPN C0603C104K8RACTU -> (none); OCTOPART_URL https://octopart.com/c0603c104k8ractu-kemet-145075?r=sp&s=9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 -> (none); TOLERANCE 10% -> (none); VOLTAGE_RATING 10 -> (none)
- C6: value ESH477M035AH3AA -> 4.7uF; device HEXABITZ_RCLS:ESH477M035AH3AA -> HEXABITZ_RCLS:C-0603-POL; CAPACITANCE 470uF -> 4.7uF; MFN (none) -> Murata; MPN (none) -> GRM21BC81E475KA12L; OCTOPART_URL (none) -> https://octopart.com/grm21bc81e475ka12l-murata-10331911?r=s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; TOLERANCE (none) -> 10%; VOLTAGE_RATING (none) -> 25V; VOLT_RATING 35V -> (none)
- C7: value 4.7uF -> 100nF; device HEXABITZ_RCLS:C-0603-POL -> HEXABITZ_RCLS:C-0402; CAPACITANCE 4.7uF -> 100nF; MFN Murata -> KEMET; MPN GRM21BC81E475KA12L -> C0603C104K8RACTU; OCTOPART_URL https://octopart.com/grm21bc81e475ka12l-murata-10331911?r=s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 -> https://octopart.com/c0603c104k8ractu-kemet-145075?r=sp&s=9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; VOLTAGE_RATING 25V -> 10V
- C8: value 100nF -> (none); MFN KEMET -> (none); MPN C0603C104K8RACTU -> (none); OCTOPART_URL https://octopart.com/c0603c104k8ractu-kemet-145075?r=sp&s=9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 -> (none); TOLERANCE 10% -> (none); VOLTAGE_RATING 10V -> 50V
- D1: device HEXABITZ_USER_INTERFACE_PARTS:VLMS1300-GS08 -> Hexabitz:VLMS1300-GS08
- D2: value ORANGE -> BOURNS_CDSOD323-T03SCBOURNS_CDSOD323-T03SC_0_0; device HEXABITZ_USER_INTERFACE_PARTS:VLMS1300-GS08 -> HEXABITZ_RCLS:BOURNS_CDSOD323-T03SCBOURNS_CDSOD323-T03SC_0_0; MFN Vishay -> (none); MPN VLMO1300-GS08 -> (none); OCTOPART_URL https://octopart.com/vlmo1300-gs08-vishay-21709200?r=sp# -> (none)
- FB1: value FB-TDK_MMZ1608Y300B -> (none); device HEXABITZ_RCLS:FB-TDK_MMZ1608Y300B -> HEXABITZ_RCLS:FB-0603; MFN TDK -> (none); MPN MMZ1608Y300B -> (none); OCTOPART_URL https://octopart.com/mmz1608y300b-tdk-368280?r=sp&s=cd9_2ZE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 -> (none)
- R1: value 270.0R -> 270R; device HEXABITZ_RCLS:R-0402 -> HEXABITZ_RCLS:R-0603; MFN Yageo -> (none); MPN RC0603FR-07270RL -> (none); OCTOPART_URL https://octopart.com/search?q=RC0603FR-07270RL&start=0 -> (none); RESISTANCE 270.0 Ohm -> (none); TOLERANCE 1% -> (none)
- R10, R13: value 10R -> 1k
- R11: value 1K -> 47
- R12: value 1K -> 10k
- R2: device HEXABITZ_RCLS:R-0402 -> HEXABITZ_RCLS:R-0603; MFN Yageo -> (none); MPN RC0603JR-070RL -> (none); OCTOPART_URL https://octopart.com/rc0603jr-070rl-yageo-1241539?r=sp&s=X2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 -> (none); RESISTANCE 0.0 Ohm -> (none)
- R3: value 10.0K -> 10k
- R4: value 1k -> 10
- R5: value 1k -> 150; POWER (none) -> 0.25W
- R6: value 10R -> 50k; MPN RC0603JR-070RL -> RC0603JR-071KL; OCTOPART_URL https://octopart.com/rc0603jr-070rl-yageo-1241539?r=sp&s=X2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 -> https://octopart.com/rc0603jr-071kl-yageo-55402888?r=sp; RESISTANCE 0.0 Ohm -> 1k; TOLERANCE (none) -> 1%
- R7: value 0.001R -> 2.5m; device HEXABITZ_RCLS:R_1206R1206 -> HEXABITZ_RCLS:R-US_R2512; MPN PA1206FRM470R01L -> (none); POWER (none) -> 1W
- R9: value 1K -> 3.3k
Connections:
- removed net +LOAD: D4.C, J1.3, R13.2, R7.2, R8.2
- removed net CS: Q2.D, R10.2, R7.1
- removed net EN_PIN: R11.2, R9.2, U1.PD1
- removed net N$10: Q2.G, R6.1
- removed net N$11: C13.1, R10.1, U2.IN+
- removed net N$12: R6.2, U3.E1/E2
- removed net N$18: C13.2, R13.1, U2.IN-
- removed net N$7: C10.2, R5.1, U3.B1/B2
- new net AGND: C5.2, C6.2, R2.2
- new net LED_INDICATOR: R1.1, U1.PA4
- new net LOAD+: D6.K, LOAD.1, Q2.D
- new net LOAD-: LOAD.2, R10.2, R7.2
- new net N$19: D3.C, D5.A, Q2.G, R14.2, R5.1
- new net N$6: C11.1, IC1.IN1+, R10.1, R6.2
- new net N$9: C10.1, IC1.IN1-, R13.1, R15.2
- new net SWITCH_CONTROL: R11.2, R9.2, U1.PA8
- new net VCC: C13.2, IC1.VCC+
- net +VS: now also C15.+, C8.2, D4.A, R14.1, SUPPLY.1; no longer C15.2, C16.2, C17.1, C6.+, J1.1
- net CURRENT_SENSE: now also C10.2, IC1.OUT1, R15.1; no longer U2.OUT
- net GND: now also C7.2, D2.C; no longer C8.2
- net N$13: now also D3.A; no longer C10.1
- net N$16: now also U3.E1/E2; no longer Q3.C, R12.1
- net N$3: now also Q3.C, R12.1, U3.B1/B2; no longer R1.2, U1.PA4
- net N$4: now also R1.2; no longer R1.1
- net N$5: now also C7.1; no longer C8.1
- net N$8: now also D4.C, D5.K; no longer D2.A, R8.1
- net VDD: now also D2.A, FB1.1; no longer FB1.2
- net VDDA: now also C6.1, FB1.2; no longer C11.1, C7.1, FB1.1, U2.V+
- net VSSA: now also C13.1, C15.-, C8.1, D6.A, IC1.VCC-, R13.2, R6.1, R7.1, SUPPLY.2; no longer C15.1, C16.1, C17.2, C5.2, C6.-, C7.2, D2.C, D4.A, J1.2, R2.2, U2.GND, U2.REF
Other:
- note added: "18V 0.5W"
- note added: "1N4148W-7-F"
- note added: "Current Sense"
- note added: "DC Switch / PWM Switch"
- note added: "Gain = 0.125 V/A 2.5V at 20A"
- note added: "Load Connector"
- note added: "Power Connector"
- note added: "VS = up to 20V"
- note removed: "Current-Shunt Monitor"
- note removed: "Driver Output Led_Ind"
- note removed: "Driver Power Coupling"
- note removed: "Gain = 100 V/V"
- note removed: "Gain = 100 V/V Gain Error = 0.89%"
- note removed: "Ibrahim Zaeiter"
- note removed: "Input Power Coupling"
- note removed: "Load driver"
- note removed: "Power and Load Connector"
- note removed: "SPST MOSFET Switch 20A 18V"
- note removed: "U2 Coupling"
- note removed: "VS=(3.3-18) Volts"
- moved on the sheet: C1, C10, C11, C12, C13, C14, C2, C3, C4, C5, C9, D1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

Commit message: Design modification
Parts:
- C12, C8, C9: VOLTAGE_RATING 50V -> 35V
- C2: value 1.00uF -> 1uF
- R6, R8: value 50k -> 49.9k
- renumbered IC1 to U2, P2 to P1, Q3 to Q1, R15 to R8
Connections:
- removed net AGND: C5.2, C6.2, R2.2
- net VSSA: now also C5.2, C6.2, R2.2
Other:
- note added: "I_Load = up to 20A"
- note added: "check footprint"
- moved on the sheet: C7, R3, RESET, SWD, X1

Commit message: Schematic modification
Parts:
- added R15: 100k, HEXABITZ_RCLS:R-0402
Connections:
- net N$14: now also R15.1
- net VSSA: now also R15.2
Other:
- moved on the sheet: C14, Q1, R11, R12, R9
Changed lines of the file:
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@@
 <part name="SUPPLY18" library="supply2" deviceset="VDD" device=""/>
 <part name="SUPPLY19" library="HEXABITZ_CONNECTION_PARTS" library_urn="urn:adsk.eagle:library:20064553" deviceset="VSSA" device=""/>
+<part name="R15" library="HEXABITZ_RCLS" library_urn="urn:adsk.eagle:library:20064561" deviceset="R-0402" device="" package3d_urn="urn:adsk.eagle:package:19666455/3" value="100k">
+<attribute name="MFN" value="Yageo"/>
+<attribute name="MPN" value="RC0603JR-07680KL"/>
+<attribute name="OCTOPART_URL" value="https://octopart.com/rc0603jr-07680kl-yageo-40953169?r=sp"/>
+<attribute name="RESISTANCE" value="680K Ohm"/>
+<attribute name="TOLERANCE" value="5%"/>
+</part>
+<part name="SUPPLY21" library="HEXABITZ_CONNECTION_PARTS" library_urn="urn:adsk.eagle:library:20064553" deviceset="VSSA" device=""/>
 </parts>
 <sheets>
@@
 <attribute name="VALUE" x="249.555" y="85.09" size="1.778" layer="96" rot="R180"/>
 </instance>
-<instance part="R12" gate="G$1" x="64.77" y="135.89" smashed="yes" rot="R90">
-<attribute name="NAME" x="62.865" y="138.2014" size="1.778" layer="95" rot="R180"/>
-<attribute name="VALUE" x="62.23" y="135.382" size="1.778" layer="96" rot="R180"/>
+<instance part="R12" gate="G$1" x="69.215" y="135.89" smashed="yes" rot="R90">
+<attribute name="NAME" x="67.31" y="138.2014" size="1.778" layer="95" rot="R180"/>
+<attribute name="VALUE" x="66.675" y="135.382" size="1.778" layer="96" rot="R180"/>
 </instance>
 <instance part="R5" gate="G$1" x="120.65" y="127.635" smashed="yes" rot="R180">
@@
 <attribute name="POWER" x="124.46" y="126.365" size="1.778" layer="96" rot="R180"/>
 </instance>
-<instance part="Q1" gate="G$1" x="62.23" y="119.38" smashed="yes">
-<attribute name="NAME" x="60.96" y="123.825" size="1.778" layer="95"/>
-<attribute name="VALUE" x="66.04" y="127.635" size="1.778" layer="96" rot="R270"/>
+<instance part="Q1" gate="G$1" x="66.675" y="119.38" smashed="yes">
+<attribute name="NAME" x="65.405" y="123.825" size="1.778" layer="95"/>
+<attribute name="VALUE" x="70.485" y="127.635" size="1.778" layer="96" rot="R270"/>
 </instance>
 <instance part="U3" gate="A" x="91.44" y="125.73" smashed="yes">
@@
 <attribute name="VALUE" x="116.84" y="140.843" size="1.778" layer="96"/>
 </instance>
-<instance part="R9" gate="G$1" x="49.53" y="119.38" smashed="yes" rot="R180">
-<attribute name="NAME" x="48.26" y="121.5136" size="1.778" layer="95"/>
-<attribute name="VALUE" x="47.625" y="116.078" size="1.778" layer="96"/>
-</instance>
-<instance part="C14" gate="G$1" x="55.245" y="128.27" smashed="yes" rot="R90">
-<attribute name="NAME" x="56.261" y="132.969" size="1.778" layer="95" rot="R180"/>
-<attribute name="VALUE" x="56.261" y="125.349" size="1.778" layer="96" rot="R180"/>
-</instance>
-<instance part="R11" gate="G$1" x="44.45" y="128.27" smashed="yes" rot="R180">
-<attribute name="NAME" x="41.91" y="131.0386" size="1.778" layer="95"/>
-<attribute name="VALUE" x="42.545" y="123.698" size="1.778" layer="96"/>
+<instance part="R9" gate="G$1" x="52.07" y="119.38" smashed="yes" rot="R180">
+<attribute name="NAME" x="50.8" y="121.5136" size="1.778" layer="95"/>
+<attribute name="VALUE" x="50.165" y="116.078" size="1.778" layer="96"/>
+</instance>
+<instance part="C14" gate="G$1" x="57.785" y="128.27" smashed="yes" rot="R90">
+<attribute name="NAME" x="58.801" y="132.969" size="1.778" layer="95" rot="R180"/>
+<attribute name="VALUE" x="58.801" y="125.349" size="1.778" layer="96" rot="R180"/>
+</instance>
+<instance part="R11" gate="G$1" x="46.99" y="128.27" smashed="yes" rot="R180">
+<attribute name="NAME" x="44.45" y="131.0386" size="1.778" layer="95"/>
+<attribute name="VALUE" x="45.085" y="123.698" size="1.778" layer="96"/>
 </instance>
 <instance part="P+1" gate="1" x="15.875" y="198.755" smashed="yes">
@@
 <attribute name="VALUE" x="161.925" y="187.96" size="1.778" layer="96" rot="R180"/>
 </instance>
-<instance part="SUPPLY12" gate="G$1" x="64.77" y="102.87" smashed="yes">
-<attribute name="VALUE" x="61.468" y="99.06" size="1.778" layer="96"/>
+<instance part="SUPPLY12" gate="G$1" x="69.215" y="102.87" smashed="yes">
+<attribute name="VALUE" x="65.913" y="99.06" size="1.778" layer="96"/>
 </instance>
 <instance part="C15" gate="G$1" x="167.64" y="179.705" smashed="yes" rot="R270">
@@
 <attribute name="VALUE" x="110.49" y="157.48" size="1.778" layer="96" rot="R180"/>
 </instance>
-<instance part="P+4" gate="1" x="64.77" y="145.415" smashed="yes">
-<attribute name="VALUE" x="67.31" y="149.225" size="1.778" layer="96" rot="R180"/>
+<instance part="P+4" gate="1" x="69.215" y="145.415" smashed="yes">
+<attribute name="VALUE" x="71.755" y="149.225" size="1.778" layer="96" rot="R180"/>
 </instance>
 <instance part="SUPPLY19" gate="G$1" x="167.64" y="162.56" smashed="yes">
 <attribute name="VALUE" x="164.338" y="158.75" size="1.778" layer="96"/>
 </instance>
+<instance part="R15" gate="G$1" x="60.96" y="111.76" smashed="yes" rot="R270">
+<attribute name="NAME" x="62.865" y="111.9886" size="1.778" layer="95"/>
+<attribute name="VALUE" x="62.865" y="109.728" size="1.778" layer="96"/>
+</instance>
+<instance part="SUPPLY21" gate="G$1" x="60.96" y="102.87" smashed="yes">
+<attribute name="VALUE" x="57.658" y="99.06" size="1.778" layer="96"/>
+</instance>
 </instances>
 <busses>
@@
 <segment>
 <pinref part="R9" gate="G$1" pin="1"/>
-<wire x1="54.61" y1="119.38" x2="58.42" y2="119.38" width="0.1524" layer="91"/>
+<wire x1="57.15" y1="119.38" x2="60.96" y2="119.38" width="0.1524" layer="91"/>
 <pinref part="Q1" gate="G$1" pin="B"/>
-<wire x1="59.69" y1="119.38" x2="58.42" y2="119.38" width="0.1524" layer="91"/>
+<wire x1="64.135" y1="119.38" x2="60.96" y2="119.38" width="0.1524" layer="91"/>
 <pinref part="C14" gate="G$1" pin="2"/>
-<wire x1="57.785" y1="128.27" x2="58.42" y2="128.27" width="0.1524" layer="91"/>
-<wire x1="58.42" y1="128.27" x2="58.42" y2="119.38" width="0.1524" layer="91"/>
-<junction x="58.42" y="119.38"/>
+<wire x1="60.325" y1="128.27" x2="60.96" y2="128.27" width="0.1524" layer="91"/>
+<wire x1="60.96" y1="128.27" x2="60.96" y2="119.38" width="0.1524" layer="91"/>
+<junction x="60.96" y="119.38"/>
+<pinref part="R15" gate="G$1" pin="1"/>
+<wire x1="60.96" y1="116.84" x2="60.96" y2="119.38" width="0.1524" layer="91"/>
 </segment>
 </net>
@@
 <pinref part="R11" gate="G$1" pin="1"/>
 <pinref part="C14" gate="G$1" pin="1"/>
-<wire x1="49.53" y1="128.27" x2="50.165" y2="128.27" width="0.1524" layer="91"/>
+<wire x1="52.07" y1="128.27" x2="52.705" y2="128.27" width="0.1524" layer="91"/>
 </segment>
 </net>
@@
 <segment>
 <pinref part="R11" gate="G$1" pin="2"/>
-<wire x1="39.37" y1="128.27" x2="38.735" y2="128.27" width="0.1524" layer="91"/>
-<wire x1="38.735" y1="128.27" x2="38.735" y2="119.38" width="0.1524" layer="91"/>
-<label x="37.465" y="119.38" size="1.778" layer="95" rot="MR0" xref="yes"/>
+<wire x1="41.91" y1="128.27" x2="41.275" y2="128.27" width="0.1524" layer="91"/>
+<wire x1="41.275" y1="128.27" x2="41.275" y2="119.38" width="0.1524" layer="91"/>
+<label x="40.005" y="119.38" size="1.778" layer="95" rot="MR0" xref="yes"/>
 <pinref part="R9" gate="G$1" pin="2"/>
-<wire x1="38.735" y1="119.38" x2="37.465" y2="119.38" width="0.1524" layer="91"/>
-<wire x1="44.45" y1="119.38" x2="38.735" y2="119.38" width="0.1524" layer="91"/>
-<junction x="38.735" y="119.38"/>
+<wire x1="41.275" y1="119.38" x2="40.005" y2="119.38" width="0.1524" layer="91"/>
+<wire x1="46.99" y1="119.38" x2="41.275" y2="119.38" width="0.1524" layer="91"/>
+<junction x="41.275" y="119.38"/>
 </segment>
 </net>
@@
 <segment>
 <pinref part="R12" gate="G$1" pin="2"/>
-<wire x1="64.77" y1="140.97" x2="64.77" y2="142.875" width="0.1524" layer="91"/>
+<wire x1="69.215" y1="140.97" x2="69.215" y2="142.875" width="0.1524" layer="91"/>
 <pinref part="P+4" gate="1" pin="+VS"/>
 </segment>
@@
 <pinref part="Q1" gate="G$1" pin="E"/>
 <pinref part="SUPPLY12" gate="G$1" pin="VSSA"/>
-<wire x1="64.77" y1="114.3" x2="64.77" y2="105.41" width="0.1524" layer="91"/>
+<wire x1="69.215" y1="114.3" x2="69.215" y2="105.41" width="0.1524" layer="91"/>
 </segment>
 <segment>
@@
 <wire x1="167.64" y1="165.1" x2="167.64" y2="167.005" width="0.1524" layer="91"/>
 </segment>
+<segment>
+<pinref part="R15" gate="G$1" pin="2"/>
+<pinref part="SUPPLY21" gate="G$1" pin="VSSA"/>
+<wire x1="60.96" y1="106.68" x2="60.96" y2="105.41" width="0.1524" layer="91"/>
+</segment>
 </net>
 <net name="N$16" class="0">
@@
 <pinref part="Q1" gate="G$1" pin="C"/>
 <pinref part="R12" gate="G$1" pin="1"/>
-<wire x1="64.77" y1="130.81" x2="64.77" y2="128.27" width="0.1524" layer="91"/>
+<wire x1="69.215" y1="130.81" x2="69.215" y2="128.27" width="0.1524" layer="91"/>
 <pinref part="U3" gate="A" pin="B1/B2"/>
-<wire x1="64.77" y1="128.27" x2="64.77" y2="124.46" width="0.1524" layer="91"/>
-<wire x1="76.2" y1="128.27" x2="64.77" y2="128.27" width="0.1524" layer="91"/>
-<junction x="64.77" y="128.27"/>
+<wire x1="69.215" y1="128.27" x2="69.215" y2="124.46" width="0.1524" layer="91"/>
+<wire x1="76.2" y1="128.27" x2="69.215" y2="128.27" width="0.1524" layer="91"/>
+<junction x="69.215" y="128.27"/>
 </segment>
 </net>

Commit message: -Edit the description
Other:
- note added: "20V 20A DC Switch / PWM Switch"
- note added: "Note! check footprint"
- note removed: "DC Switch / PWM Switch"
- note removed: "check footprint"
Changed lines of the file:
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@@
 <wire x1="231.14" y1="18.288" x2="231.14" y2="22.86" width="0.1524" layer="205"/>
 <text x="242.6462" y="6.1722" size="1.9304" layer="100" font="vector">www.hexabitz.com</text>
-<text x="179.2478" y="11.2014" size="1.9304" layer="101" font="vector">DC Switch / PWM Switch</text>
+<text x="170.9928" y="11.2014" size="1.9304" layer="101" font="vector">20V 20A DC Switch / PWM Switch</text>
 <text x="137.71" y="95.455" size="1.778" layer="95">VDDA Coupling</text>
 </plain>
@@
 <wire x1="231.14" y1="18.288" x2="231.14" y2="22.86" width="0.1524" layer="205"/>
 <text x="242.6462" y="6.1722" size="1.9304" layer="100" font="vector">www.hexabitz.com</text>
-<text x="177.9778" y="11.2014" size="1.9304" layer="101" font="vector">DC Switch / PWM Switch</text>
+<text x="172.2628" y="11.2014" size="1.9304" layer="101" font="vector">20V 20A DC Switch / PWM Switch</text>
 <text x="146.05" y="143.51" size="1.778" layer="91">1N4148W-7-F</text>
 <text x="210.82" y="48.26" size="2.54" layer="89" font="vector" ratio="11" distance="46">Gain = 0.125 V/A
@@
 <text x="132.715" y="143.51" size="1.778" layer="91">18V 0.5W</text>
 <text x="212.725" y="104.775" size="2.54" layer="89" font="vector" ratio="11" distance="46">I_Load = up to 20A</text>
-<text x="130.175" y="156.21" size="1.778" layer="91">check footprint</text>
+<text x="126.365" y="156.21" size="1.778" layer="91">Note! check footprint</text>
 </plain>
 <instances>
